File: PCB_Relay/Arduino-Pro-Mini.brd (EAGLE design)
At the start: 17.8 x 33 mm, 30 parts, among them T1 BC547, T2 BC547, T3 BC547, T4 BC547

Commit message: board file small change .
Routing:
- net A1: track 52.2 -> 53.7 mm
Changed lines of the file:
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@@
 <layer number="16" name="Bottom" color="1" fill="1" visible="yes" active="yes"/>
 <layer number="17" name="Pads" color="2" fill="1" visible="yes" active="yes"/>
-<layer number="18" name="Vias" color="2" fill="1" visible="no" active="yes"/>
+<layer number="18" name="Vias" color="2" fill="1" visible="yes" active="yes"/>
 <layer number="19" name="Unrouted" color="6" fill="1" visible="yes" active="yes"/>
 <layer number="20" name="Dimension" color="6" fill="1" visible="no" active="yes"/>
 <layer number="21" name="tPlace" color="16" fill="1" visible="yes" active="yes"/>
-<layer number="22" name="bPlace" color="14" fill="1" visible="no" active="yes"/>
+<layer number="22" name="bPlace" color="14" fill="1" visible="yes" active="yes"/>
 <layer number="23" name="tOrigins" color="15" fill="1" visible="yes" active="yes"/>
 <layer number="24" name="bOrigins" color="15" fill="1" visible="yes" active="yes"/>
@@
 <contactref element="T2" pad="2"/>
 <contactref element="R1" pad="1"/>
-<wire x1="31.51635" y1="43.95515625" x2="35.395" y2="48.145" width="0.4064" layer="16"/>
-<wire x1="31.51635" y1="43.95515625" x2="31.095" y2="43.5" width="0.4064" layer="16"/>
-<wire x1="35.395" y1="48.145" x2="34.34" y2="51" width="0.4064" layer="16"/>
+<wire x1="31.095" y1="43.5" x2="31.51635" y2="43.95515625" width="0.4064" layer="16"/>
 <wire x1="17.3" y1="14.2" x2="18.3" y2="13.2" width="0.4064" layer="16"/>
 <wire x1="17.3" y1="14.2" x2="16.74" y2="14.2" width="0.4064" layer="16"/>
@@
 <wire x1="31.1" y1="35.2" x2="31.1" y2="43.53880625" width="0.254" layer="16"/>
 <wire x1="31.1" y1="43.53880625" x2="31.51635" y2="43.95515625" width="0.254" layer="16"/>
+<wire x1="34.34" y1="51" x2="32.8" y2="51" width="0.4064" layer="16"/>
+<wire x1="32.8" y1="51" x2="31.4" y2="49.6" width="0.4064" layer="16"/>
+<wire x1="31.4" y1="49.6" x2="31.4" y2="47.1" width="0.4064" layer="16"/>
+<wire x1="31.4" y1="47.1" x2="30.4" y2="46.1" width="0.4064" layer="16"/>
+<wire x1="30.4" y1="46.1" x2="30.4" y2="44.195" width="0.4064" layer="16"/>
+<wire x1="30.4" y1="44.195" x2="31.095" y2="43.5" width="0.4064" layer="16"/>
 </signal>
 <signal name="A0">
